File: circuito/rasp-sense33/trekking.kicad_pcb (KiCad board)
At the start: 2 copper layers, 100 x 100 mm, 7 parts, among them J1 Raspberry Pi, U1 RPI-PICO

Commit message: driver motor rev 2
Parts:
- added C1: 100nF, Capacitor_SMD:C_0805_2012Metric_Pad1.18x1.45mm_HandSolder, F.Cu at (129.4, 33.5)
- added C2: 100nF, Capacitor_SMD:C_0805_2012Metric_Pad1.18x1.45mm_HandSolder, F.Cu at (139.0, 34.6)
- added C3: 10uF6V3, Capacitor_SMD:C_0805_2012Metric_Pad1.18x1.45mm_HandSolder, F.Cu at (134.2, 34.6)
- added J10: MOTOR, Connector_Molex:Molex_KK-254_AE-6410-04A_1x04_P2.54mm_Vertical, F.Cu at (128.5, 134.5)
- added J11: OUT, MyFootprint:CONN5mm-3, F.Cu at (45.0, 71.0)
- added J12: I2C0, Connector_Molex:Molex_KK-254_AE-6410-04A_1x04_P2.54mm_Vertical, F.Cu at (85.5, 138.5)
- added J13: I2C0, Connector_Molex:Molex_KK-254_AE-6410-04A_1x04_P2.54mm_Vertical, F.Cu at (85.5, 114.5)
- added J14: I2C0, Connector_Molex:Molex_KK-254_AE-6410-04A_1x04_P2.54mm_Vertical, F.Cu at (85.5, 130.5)
- added J15: I2C0, Connector_Molex:Molex_KK-254_AE-6410-04A_1x04_P2.54mm_Vertical, F.Cu at (85.5, 106.5)
- added J16: I2C0, Connector_Molex:Molex_KK-254_AE-6410-04A_1x04_P2.54mm_Vertical, F.Cu at (85.5, 122.5)
- added J17: I2C0, Connector_Molex:Molex_KK-254_AE-6410-04A_1x04_P2.54mm_Vertical, F.Cu at (85.5, 98.5)
- added J18: Module, Connector_PinHeader_2.54mm:PinHeader_1x08_P2.54mm_Vertical, F.Cu at (120.5, 72.6)
- added J19: OUT, MyFootprint:CONN5mm-3, F.Cu at (45.0, 86.0)
- added J2: ENCODER, Connector_Molex:Molex_KK-254_AE-6410-04A_1x04_P2.54mm_Vertical, F.Cu at (128.5, 114.5)
- added J20: OUT, MyFootprint:CONN5mm-3, F.Cu at (45.0, 101.0)
- added J21: INPUT, MyFootprint:CONN5mm-3, F.Cu at (45.0, 131.0)
- added J22: INPUT, MyFootprint:CONN5mm-3, F.Cu at (45.0, 116.0)
- added J3: ENCODER, Connector_Molex:Molex_KK-254_AE-6410-04A_1x04_P2.54mm_Vertical, F.Cu at (128.5, 122.5)
- added J4: ENCODER, Connector_Molex:Molex_KK-254_AE-6410-04A_1x04_P2.54mm_Vertical, F.Cu at (128.5, 98.5)
- added J5: ENCODER, Connector_Molex:Molex_KK-254_AE-6410-04A_1x04_P2.54mm_Vertical, F.Cu at (128.5, 106.5)
- added J6: VIN, MyFootprint:AK300-2, F.Cu at (133.0, 73.0)
- added J7: VCC, MyFootprint:AK300-2, F.Cu at (122.2, 62.0)
- added J8: 5VIN, MyFootprint:AK300-2, F.Cu at (112.0, 62.0)
- added J9: MOTOR, Connector_Molex:Molex_KK-254_AE-6410-04A_1x04_P2.54mm_Vertical, F.Cu at (128.5, 142.5)
- added R1: 10K, Resistor_SMD:R_0805_2012Metric_Pad1.20x1.40mm_HandSolder, F.Cu at (148.5, 34.6)
- added R10: 10K, Resistor_SMD:R_0805_2012Metric_Pad1.20x1.40mm_HandSolder, F.Cu at (51.0, 141.0)
- added R11: 10K, Resistor_SMD:R_0805_2012Metric_Pad1.20x1.40mm_HandSolder, F.Cu at (51.0, 116.0)
- added R12: 10K, Resistor_SMD:R_0805_2012Metric_Pad1.20x1.40mm_HandSolder, F.Cu at (51.0, 121.0)
- added R13: 10K, Resistor_SMD:R_0805_2012Metric_Pad1.20x1.40mm_HandSolder, F.Cu at (51.0, 126.0)
- added R14: 1K, Resistor_SMD:R_0805_2012Metric_Pad1.20x1.40mm_HandSolder, F.Cu at (51.0, 133.5)
- added R15: 1K, Resistor_SMD:R_0805_2012Metric_Pad1.20x1.40mm_HandSolder, F.Cu at (51.0, 138.2)
- added R16: 1K, Resistor_SMD:R_0805_2012Metric_Pad1.20x1.40mm_HandSolder, F.Cu at (51.0, 143.4)
- added R17: 1K, Resistor_SMD:R_0805_2012Metric_Pad1.20x1.40mm_HandSolder, F.Cu at (51.0, 118.5)
- added R18: 1K, Resistor_SMD:R_0805_2012Metric_Pad1.20x1.40mm_HandSolder, F.Cu at (51.0, 123.5)
- added R19: 1K, Resistor_SMD:R_0805_2012Metric_Pad1.20x1.40mm_HandSolder, F.Cu at (51.0, 128.0)
- added R2: 1K, Resistor_SMD:R_0805_2012Metric_Pad1.20x1.40mm_HandSolder, F.Cu at (129.2, 42.6)
- added R3: ~0., Resistor_SMD:R_1206_3216Metric_Pad1.30x1.75mm_HandSolder, F.Cu at (124.0, 33.6)
- added R4: 10K, Resistor_SMD:R_0805_2012Metric_Pad1.20x1.40mm_HandSolder, F.Cu at (128.2, 45.6)
- added R5: 1K, Resistor_SMD:R_0805_2012Metric_Pad1.20x1.40mm_HandSolder, F.Cu at (123.2, 44.6)
- added R6: 10K, Resistor_SMD:R_0805_2012Metric_Pad1.20x1.40mm_HandSolder, F.Cu at (135.2, 45.6)
- added R7: 1K, Resistor_SMD:R_0805_2012Metric_Pad1.20x1.40mm_HandSolder, F.Cu at (143.8, 34.6)
- added R8: 10K, Resistor_SMD:R_0805_2012Metric_Pad1.20x1.40mm_HandSolder, F.Cu at (51.0, 131.0)
- added R9: 10K, Resistor_SMD:R_0805_2012Metric_Pad1.20x1.40mm_HandSolder, F.Cu at (51.0, 136.0)
- added U2: AMS1117-3.3, Package_TO_SOT_SMD:SOT-223-3_TabPin2, F.Cu at (114.2, 37.6)
- added U3: ULN2803A, Package_SO:SOIC-18W_7.5x11.6mm_P1.27mm, F.Cu at (71.2, 108.1)
- U1: footprint trekking-library:RPI_PICO -> MyFootprint:RPI-PICO-SMD
- moved U1 62.6 mm to (119.0, 95.1)
- moved A1 24.3 mm to (63.6, 106.1)
- moved J1 4.49 mm to (54.4, 64.3)
Connections:
- A1 pad 1: unconnected-(A1-Pad1) -> /TX
- A1 pad 10: unconnected-(A1-Pad10) -> /D7
- A1 pad 11: unconnected-(A1-Pad11) -> /D8
- A1 pad 12: unconnected-(A1-Pad12) -> /D9
- A1 pad 13: unconnected-(A1-Pad13) -> /SC
- A1 pad 14: unconnected-(A1-Pad14) -> /MOSI
- A1 pad 15: unconnected-(A1-Pad15) -> /MISO
- A1 pad 16: unconnected-(A1-Pad16) -> /SCK
- A1 pad 19: unconnected-(A1-Pad19) -> /A0
- A1 pad 2: unconnected-(A1-Pad2) -> /RX
- A1 pad 20: unconnected-(A1-Pad20) -> /A1
- A1 pad 21: unconnected-(A1-Pad21) -> /A2
- A1 pad 22: unconnected-(A1-Pad22) -> /A3
- A1 pad 25: unconnected-(A1-Pad25) -> /A6
- A1 pad 26: unconnected-(A1-Pad26) -> /A7
- A1 pad 5: unconnected-(A1-Pad5) -> /D2
- A1 pad 6: unconnected-(A1-Pad6) -> /D3
- A1 pad 7: unconnected-(A1-Pad7) -> /D4
- A1 pad 8: unconnected-(A1-Pad8) -> /D5
- A1 pad 9: unconnected-(A1-Pad9) -> /D6
- J1 pad 19: unconnected-(J1-Pad19) -> /MOSI
- J1 pad 21: unconnected-(J1-Pad21) -> /MISO
- J1 pad 23: unconnected-(J1-Pad23) -> /SCK
- J1 pad 24: unconnected-(J1-Pad24) -> /SC
- U1 pad 41: Earth -> /SWCLK
- U1 pad 42: (no net) -> Earth
- U1 pad 43: (no net) -> /SWDIO
Routing:
- net +3V3: track 0.00 -> 157.9 mm
- net /SCL0: track 0.00 -> 149.6 mm, vias 0 -> 1
- net /SDA0: track 0.00 -> 142.5 mm, vias 0 -> 1
- net /TXD0: track 0.00 -> 139.5 mm
- net /RXD0: track 0.00 -> 138.5 mm
- net /SC: track 0.00 -> 122.1 mm
- net +5V: track 0.00 -> 99.4 mm
- net /MISO: track 0.00 -> 84.1 mm
- net /SCK: track 0.00 -> 84.0 mm
- net /MOSI: track 0.00 -> 80.5 mm
- net /A7: track 0.00 -> 71.8 mm
- net /A6: track 0.00 -> 65.5 mm
- net /A3: track 0.00 -> 55.6 mm
- net /A2: track 0.00 -> 50.8 mm
- net /O9: track 0.00 -> 46.2 mm
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
Commit message: driver motor rev 2
Parts:
- removed C1: 100nF, Capacitor_SMD:C_0805_2012Metric_Pad1.18x1.45mm_HandSolder
- removed U2: AMS1117-3.3, Package_TO_SOT_SMD:SOT-223-3_TabPin2
- added J23: ENCODER, Connector_Molex:Molex_KK-254_AE-6410-04A_1x04_P2.54mm_Vertical, F.Cu at (85.5, 151.0)
- added VCC: TestPoint_THTPad_D1.5mm_Drill0.7mm, TestPoint:TestPoint_THTPad_D1.5mm_Drill0.7mm, F.Cu at (121.0, 76.5)
- added VIN: TestPoint_THTPad_D1.5mm_Drill0.7mm, TestPoint:TestPoint_THTPad_D1.5mm_Drill0.7mm, F.Cu at (121.0, 82.0)
- moved R7 112.0 mm to (82.0, 128.0), turned to 90 degrees
- moved R6 104.5 mm to (82.0, 135.5), turned to 90 degrees
- moved R1 55.9 mm to (123.5, 84.5), turned to 180 degrees
- moved R3 45.4 mm to (124.5, 79.0), turned to 90 degrees
- moved R2 44.8 mm to (123.5, 87.0)
- moved C2 33.7 mm to (118.0, 61.0), turned to 90 degrees
- moved C3 32.6 mm to (115.0, 61.0), turned to 90 degrees
- moved R4 28.8 mm to (123.5, 74.0), turned to 180 degrees
- moved R5 27.3 mm to (123.5, 71.9)
- moved J7 16.2 mm to (133.0, 74.1), turned to -90 degrees
- moved J6 11.2 mm to (133.0, 84.2)
- moved J8 10.5 mm to (122.5, 62.0)
- moved J18 8.17 mm to (113.0, 69.4)
Connections:
- A1 pad 1: /TX -> /ATX
- A1 pad 2: /RX -> /ARX
- A1 pad 28: /RST_A -> unconnected-(A1-Pad28)
- C2 pad 1: +3V3 -> +5V
- C3 pad 1: +3V3 -> +5V
- J1 pad 26: unconnected-(J1-Pad26) -> /RST_A
- J1 pad 29: /G22 -> unconnected-(J1-Pad29)
- J1 pad 33: /RST_A -> /G22
- J18 pad 7: /TXD1 -> /RXD1
- J18 pad 8: /RXD1 -> /TXD1
- J4 pad 2: /P3D -> /P3C
- J5 pad 2: /P3C -> /P3D
Routing:
- net +5V: track 99.4 -> 229.9 mm, vias 0 -> 1
- net /RST_A: track 0.00 -> 98.8 mm
- net /ATX: track 0.00 -> 82.9 mm
- net /ARX: track 0.00 -> 80.5 mm
- net /ADC1: track 0.00 -> 69.7 mm, vias 0 -> 2
- net /ADC2: track 0.00 -> 63.1 mm, vias 0 -> 2
- net /G22: track 0.00 -> 57.9 mm
- net /RUN: track 0.00 -> 57.7 mm
- net /P3D: track 0.00 -> 38.1 mm, vias 0 -> 1
- net /P3C: track 0.00 -> 37.8 mm, vias 0 -> 1
- net /SPI0_TX: track 0.00 -> 36.8 mm, vias 0 -> 1
- net /SPI0_SCK: track 0.00 -> 36.7 mm, vias 0 -> 1
- net /RXD1: track 0.00 -> 35.3 mm
- net /TXD1: track 0.00 -> 35.2 mm
- net /SWCLK: track 27.4 -> 62.4 mm
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
Commit message: driver rasp-sense33
Parts:
- added ?: , , F.Cu at (83.0, 70.5)
- added C1: 100nF, Capacitor_SMD:C_0805_2012Metric_Pad1.18x1.45mm_HandSolder, F.Cu at (100.0, 73.0)
- added C4: 100uF50V, Capacitor_SMD:CP_Elec_8x10, F.Cu at (92.0, 72.0)
- added C5: 220uF35V, Capacitor_SMD:CP_Elec_8x10, F.Cu at (67.0, 82.0)
- added C6: 100nF, Capacitor_SMD:C_0805_2012Metric_Pad1.18x1.45mm_HandSolder, F.Cu at (60.5, 84.0)
- added D1: 1N5822, MyFootprint:My_D_MELF-RM10_Universal_Handsoldering_2, F.Cu at (66.5, 73.5)
- added L1: 33uH, Inductor_SMD:L_12x12mm_H8mm, F.Cu at (79.6, 81.0)
- added U2: LM2596T-5, Package_TO_SOT_SMD:TO-263-5_TabPin3, F.Cu at (96.0, 83.0)
- J18: footprint Connector_PinHeader_2.54mm:PinHeader_1x08_P2.54mm_Vertical -> Connector_PinHeader_2.54mm:PinHeader_1x12_P2.54mm_Vertical
- J23: value ENCODER -> UART
- moved J18 26.5 mm to (101.0, 93.0), turned to -90 degrees
- moved R3 6.50 mm to (118.0, 79.0)
- moved R1 1.25 mm to (123.5, 83.2), turned to -90 degrees
Connections:
- J1 pad 31: /RUN -> unconnected-(J1-Pad31)
- J1 pad 33: /G22 -> unconnected-(J1-Pad33)
- J1 pad 35: unconnected-(J1-Pad35) -> /G22
- J1 pad 37: unconnected-(J1-Pad37) -> /RUN
- J18 pad 1: Vmod -> /TXD1
- J18 pad 2: Earth -> /RXD1
- J18 pad 7: /RXD1 -> +3V3
- J18 pad 8: /TXD1 -> Earth
- U3 pad 10: +5V -> /VCC
Routing:
- net /VCC: track 33.8 -> 126.3 mm, vias 0 -> 3
- net /SPI0_RX: track 33.7 -> 4.39 mm, vias 1 -> 0
- net /SCK: track 84.0 -> 112.3 mm
- net /SPI0_SC: track 34.0 -> 8.99 mm, vias 1 -> 0
- net /MISO: track 84.1 -> 108.6 mm
- net /MOSI: track 80.5 -> 103.4 mm
- net Net-(D1-Pad1): track 0.00 -> 22.0 mm
- net /SPI0_SCK: track 36.7 -> 15.1 mm, vias 1 -> 0
- net +5V: track 229.9 -> 247.0 mm, vias 1 -> 2
- net /SPI0_TX: track 36.8 -> 21.2 mm
- net /SCL0: track 156.4 -> 169.3 mm
- net /RXD1: track 35.3 -> 48.0 mm, vias 0 -> 1
- net /SDA0: track 150.6 -> 162.1 mm
- net +3V3: track 167.2 -> 178.6 mm
- net /TXD1: track 35.2 -> 45.1 mm, vias 0 -> 1
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Other:
- board text added: "10"
- board text added: "11"
- board text added: "11RST"
- board text added: "12"
- board text added: "13"
- board text added: "14"
- board text added: "15"
- board text added: "16"
- board text added: "17"
- board text added: "18"
- board text added: "19"
- board text added: "2"
- board text added: "20"
- board text added: "21"
- board text added: "22 24"
- board text added: "3"
- board text added: "3V3"
- board text added: "5V"
- board text added: "6"
- board text added: "7"
- board text added: "A0"
- board text added: "A1"
- board text added: "A2"
- board text added: "A3"
- board text added: "A6"
- board text added: "A7"
- board text added: "ARX"
- board text added: "ATX"
- board text added: "D2"
- board text added: "D3"
- board text added: "D4"
- board text added: "D5"
- board text added: "D6"
- board text added: "D7"
- board text added: "D8"
- board text added: "D9"
- board text added: "G"
- board text added: "GND"
- board text added: "MISO"
- board text added: "MOSI"
- board text added: "RUN 25"
- board text added: "RX0"
- board text added: "RX1"
- board text added: "SC"
- board text added: "SCA"
- board text added: "SCK"
- board text added: "SCL"
- board text added: "SDA"
- board text added: "SWDIO"
- board text added: "SWDLK"
- board text added: "TX0"
- board text added: "TX1"
- board text added: "VCC"
- board text added: "VIN"

Commit message: incluindo movimento
Parts:
- added R20: 0, Resistor_SMD:R_0805_2012Metric_Pad1.20x1.40mm_HandSolder, B.Cu at (117.8, 72.0)
- added R21: 0, Resistor_SMD:R_0805_2012Metric_Pad1.20x1.40mm_HandSolder, B.Cu at (83.0, 81.0)
Connections:
- C1 pad 1: /VCC -> Net-(C1-Pad1)
- C4 pad 1: /VCC -> Net-(C1-Pad1)
- C5 pad 1: +5V -> Net-(C5-Pad1)
- C6 pad 1: +5V -> Net-(C5-Pad1)
- L1 pad 2: +5V -> Net-(C5-Pad1)
- U2 pad 1: /VCC -> Net-(C1-Pad1)
- U2 pad 4: +5V -> Net-(C5-Pad1)
Routing:
- net Net-(C5-Pad1): track 0.00 -> 48.3 mm, vias 0 -> 1
- net +5V: track 247.0 -> 211.8 mm, vias 2 -> 0
- net Net-(C1-Pad1): track 0.00 -> 33.2 mm, vias 0 -> 1
- net /ADC2: track 63.8 -> 58.4 mm
- net /VCC: track 126.3 -> 121.1 mm, vias 3 -> 2
- net /ADC1: track 73.2 -> 68.3 mm
- net /SCL0: track 169.3 -> 165.7 mm
- net /P3D: track 38.1 -> 35.4 mm
- net /SDA0: track 162.1 -> 160.8 mm
- net +3V3: track 178.6 -> 179.4 mm
- net /G22: track 64.3 -> 63.6 mm
- net Earth: vias 128 -> 129

Commit message: update
Routing:
- net /ADC0: track 26.3 -> 25.6 mm
- net Earth: vias 129 -> 136
Changed lines of the file:
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@@
     (pad "43" smd roundrect (at 13.412 0.017 270) (size 2.5 1.65) (layers "F.Cu" "F.Paste" "F.Mask") (roundrect_rratio 0.25)
       (net 15 "/SWDIO") (pinfunction "SWDIO") (pintype "power_in"))
+    (model "/home/pibs/workspace/Mykicad/KiCad-RP-Pico/RP-Pico Libraries/Pico.wrl"
+      (offset (xyz 10.5 25.5 0))
+      (scale (xyz 1 1 1))
+      (rotate (xyz 0 0 0))
+    )
   )
   (footprint "TestPoint:TestPoint_THTPad_D1.5mm_Drill0.7mm" (layer "F.Cu")
@@
     (pad "3" thru_hole oval locked (at 10 0 270) (size 2 4) (drill 1.5) (layers *.Cu *.Mask)
       (net 90 "Net-(J22-Pad3)") (pinfunction "Pin_3") (pintype "passive"))
+    (model "/home/pibs/workspace/Mykicad/KRE/JACK_KRE.STEP"
+      (offset (xyz 12 0 0))
+      (scale (xyz 1 1 1))
+      (rotate (xyz -90 0 90))
+    )
   )
   (footprint "Connector_Molex:Molex_KK-254_AE-6410-04A_1x04_P2.54mm_Vertical" (layer "F.Cu")
@@
     (pad "2" thru_hole rect locked (at 3.81 0 180) (size 2 2) (drill 1.19888) (layers *.Cu *.Mask)
       (net 1 "Earth") (pinfunction "A") (pintype "passive"))
-    (model "${KISYS3DMOD}/Diode_SMD.3dshapes/D_MELF.wrl"
+    (model "${KICAD6_3DMODEL_DIR}/Diode_SMD.3dshapes/D_MELF.step"
       (offset (xyz 0 0 0))
-      (scale (xyz 1 1 1))
+      (scale (xyz 1.5 1.5 1.5))
       (rotate (xyz 0 0 0))
     )
@@
     (pad "3" thru_hole oval locked (at 10 0 270) (size 2 4) (drill 1.5) (layers *.Cu *.Mask)
       (net 1 "Earth") (pinfunction "Pin_3") (pintype "passive"))
+    (model "/home/pibs/workspace/Mykicad/KRE/JACK_KRE.STEP"
+      (offset (xyz 12 0 0))
+      (scale (xyz 1 1 1))
+      (rotate (xyz -90 0 90))
+    )
   )
   (footprint "TestPoint:TestPoint_THTPad_D1.5mm_Drill0.7mm" (layer "F.Cu")
@@
     (pad "30" thru_hole oval (at 15.24 0) (size 1.6 1.6) (drill 1) (layers *.Cu *.Mask)
       (net 3 "+5V") (pinfunction "VIN") (pintype "power_in"))
-    (model "${KICAD6_3DMODEL_DIR}/Module.3dshapes/Arduino_Nano_WithMountingHoles.wrl"
+    (model "${KICAD6_3DMODEL_DIR}/Connector_PinSocket_2.54mm.3dshapes/PinSocket_1x15_P2.54mm_Vertical.wrl"
       (offset (xyz 0 0 0))
       (scale (xyz 1 1 1))
       (rotate (xyz 0 0 0))
     )
+    (model "${KICAD6_3DMODEL_DIR}/Connector_PinSocket_2.54mm.3dshapes/PinSocket_1x15_P2.54mm_Vertical.wrl"
+      (offset (xyz 15 0 0))
+      (scale (xyz 1 1 1))
+      (rotate (xyz 0 0 0))
+    )
+    (model "/home/pibs/workspace/Mykicad/Nano33BLE/Nano33BLE.step"
+      (offset (xyz 16.5 -39 10.5))
+      (scale (xyz 1 1 1))
+      (rotate (xyz 0 0 -90))
+    )
+    (model "${KICAD6_3DMODEL_DIR}/Connector_PinHeader_2.54mm.3dshapes/PinHeader_1x15_P2.54mm_Vertical.step"
+      (offset (xyz 0 0 10.05))
+      (scale (xyz 1 1 1))
+      (rotate (xyz 0 180 0))
+    )
+    (model "${KICAD6_3DMODEL_DIR}/Connector_PinHeader_2.54mm.3dshapes/PinHeader_1x15_P2.54mm_Vertical.step"
+      (offset (xyz 15 0 10.05))
+      (scale (xyz 1 1 1))
+      (rotate (xyz 0 180 0))
+    )
   )
   (footprint "Connector_Molex:Molex_KK-254_AE-6410-04A_1x04_P2.54mm_Vertical" (layer "F.Cu")
@@
     (pad "2" smd rect (at 4.95 0 270) (size 2.9 5.4) (layers "F.Cu" "F.Paste" "F.Mask")
       (net 96 "Net-(C5-Pad1)") (pinfunction "2") (pintype "passive"))
-    (model "${KICAD6_3DMODEL_DIR}/Inductor_SMD.3dshapes/L_12x12mm_H8mm.wrl"
+    (model "${KICAD6_3DMODEL_DIR}/Inductor_SMD.3dshapes/L_Bourns_SRR1260.wrl"
       (offset (xyz 0 0 0))
       (scale (xyz 1 1 1))
@@
     (pad "3" thru_hole oval locked (at 10 0 270) (size 2 4) (drill 1.5) (layers *.Cu *.Mask)
       (net 82 "/O4") (pinfunction "Pin_3") (pintype "passive"))
+    (model "/home/pibs/workspace/Mykicad/KRE/JACK_KRE.STEP"
+      (offset (xyz 12 0 0))
+      (scale (xyz 1 1 1))
+      (rotate (xyz -90 0 90))
+    )
   )
   (footprint "MyFootprint:AK300-2" (layer "F.Cu")
@@
     (pad "2" thru_hole oval (at 5 0 270) (size 2 4) (drill 1.4) (layers *.Cu *.Mask)
       (net 1 "Earth") (pinfunction "Pin_2") (pintype "passive"))
+    (model "/home/pibs/workspace/Mykicad/KRE/TBlock2vias - KRE.STEP"
+      (offset (xyz -3.4 19.05 -8.5))
+      (scale (xyz 1.2 1 1.04))
+      (rotate (xyz 90 180 90))
+    )
   )
   (footprint "Resistor_SMD:R_0805_2012Metric_Pad1.20x1.40mm_HandSolder" (layer "F.Cu")
@@
     (pad "2" thru_hole oval (at 5 0) (size 2 4) (drill 1.4) (layers *.Cu *.Mask)
       (net 1 "Earth") (pinfunction "Pin_2") (pintype "passive"))
+    (model "/home/pibs/workspace/Mykicad/KRE/TBlock2vias - KRE.STEP"
+      (offset (xyz -3.4 19.05 -8.5))
+      (scale (xyz 1.2 1 1.04))
+      (rotate (xyz 90 180 90))
+    )
   )
   (footprint "MyFootprint:CONN5mm-3" (layer "F.Cu")
@@
     (pad "3" thru_hole oval locked (at 10 0 270) (size 2 4) (drill 1.5) (layers *.Cu *.Mask)
       (net 79 "/O7") (pinfunction "Pin_3") (pintype "passive"))
+    (model "/home/pibs/workspace/Mykicad/KRE/JACK_KRE.STEP"
+      (offset (xyz 12.5 0 0))
+      (scale (xyz 1 1 1))
+      (rotate (xyz -90 0 90))
+    )
   )
   (footprint "Resistor_SMD:R_0805_2012Metric_Pad1.20x1.40mm_HandSolder" (layer "F.Cu")
@@
     (pad "3" thru_hole oval locked (at 10 0 270) (size 2 4) (drill 1.5) (layers *.Cu *.Mask)
       (net 87 "Net-(J21-Pad3)") (pinfunction "Pin_3") (pintype "passive"))
+    (model "/home/pibs/workspace/Mykicad/KRE/JACK_KRE.STEP"
+      (offset (xyz 12 0 0))
+      (scale (xyz 1 1 1))
+      (rotate (xyz -90 0 90))
+    )
   )
   (footprint "Resistor_SMD:R_0805_2012Metric_Pad1.20x1.40mm_HandSolder" (layer "F.Cu")
@@
     (pad "2" thru_hole oval (at 5 0 270) (size 2 4) (drill 1.4) (layers *.Cu *.Mask)
       (net 1 "Earth") (pinfunction "Pin_2") (pintype "passive"))
+    (model "/home/pibs/workspace/Mykicad/KRE/TBlock2vias - KRE.STEP"
+      (offset (xyz -3.4 19.05 -8.5))
+      (scale (xyz 1.2 1 1.04))
+      (rotate (xyz 90 180 90))
+    )
   )
   (footprint "Resistor_SMD:R_0805_2012Metric_Pad1.20x1.40mm_HandSolder" (layer "F.Cu")
@@
   (via (at 94.5 66.5) (size 0.8) (drill 0.4) (layers "F.Cu" "B.Cu") (free) (net 1))
   (via (at 50.8 108.8) (size 0.8) (drill 0.4) (layers "F.Cu" "B.Cu") (free) (net 1))
+  (via (at 125 66.5) (size 0.8) (drill 0.4) (layers "F.Cu" "B.Cu") (free) (net 1))
   (via (at 56 152) (size 0.8) (drill 0.4) (layers "F.Cu" "B.Cu") (free) (net 1))
   (via (at 45 78.6) (size 0.8) (drill 0.4) (layers "F.Cu" "B.Cu") (free) (net 1))
+  (via (at 135.5 76.6) (size 0.8) (drill 0.4) (layers "F.Cu" "B.Cu") (free) (net 1))
   (via (at 100.6 99.4) (size 0.8) (drill 0.4) (layers "F.Cu" "B.Cu") (free) (net 1))
   (via (at 68 70.5) (size 0.8) (drill 0.4) (layers "F.Cu" "B.Cu") (free) (net 1))
@@
   (via (at 105.5 88.5) (size 0.8) (drill 0.4) (layers "F.Cu" "B.Cu") (free) (net 1))
   (via (at 107 78.5) (size 0.8) (drill 0.4) (layers "F.Cu" "B.Cu") (free) (net 1))
+  (via (at 45 65.6) (size 0.8) (drill 0.4) (layers "F.Cu" "B.Cu") (free) (net 1))
   (via (at 67 82) (size 0.8) (drill 0.4) (layers "F.Cu" "B.Cu") (free) (net 1))
   (via (at 115.6 119.8) (size 0.8) (drill 0.4) (layers "F.Cu" "B.Cu") (free) (net 1))
@@
   (via (at 60 123.8) (size 0.8) (drill 0.4) (layers "F.Cu" "B.Cu") (free) (net 1))
   (via (at 98 76) (size 0.8) (drill 0.4) (layers "F.Cu" "B.Cu") (free) (net 1))
+  (via (at 72.8 127) (size 0.8) (drill 0.4) (layers "F.Cu" "B.Cu") (free) (net 1))
   (via (at 115.5 79) (size 0.8) (drill 0.4) (layers "F.Cu" "B.Cu") (free) (net 1))
   (via (at 107.8 101.4) (size 0.8) (drill 0.4) (layers "F.Cu" "B.Cu") (free) (net 1))
@@
   (via (at 101.8 137.4) (size 0.8) (drill 0.4) (layers "F.Cu" "B.Cu") (free) (net 1))
   (via (at 81.8 83) (size 0.8) (drill 0.4) (layers "F.Cu" "B.Cu") (free) (net 1))
-  (via (at 105 74) (size 0.8) (drill 0.4) (layers "F.Cu" "B.Cu") (free) (net 1))
+  (via (at 104.4 74.2) (size 0.8) (drill 0.4) (layers "F.Cu" "B.Cu") (free) (net 1))
   (via (at 78.8 152) (size 0.8) (drill 0.4) (layers "F.Cu" "B.Cu") (free) (net 1))
   (via (at 52.8 65.8) (size 0.8) (drill 0.4) (layers "F.Cu" "B.Cu") (free) (net 1))
@@
   (via (at 63 70.5) (size 0.8) (drill 0.4) (layers "F.Cu" "B.Cu") (free) (net 1))
   (via (at 110.4 152) (size 0.8) (drill 0.4) (layers "F.Cu" "B.Cu") (free) (net 1))
+  (via (at 135.5 81.6) (size 0.8) (drill 0.4) (layers "F.Cu" "B.Cu") (free) (net 1))
   (via (at 48.5 92) (size 0.8) (drill 0.4) (layers "F.Cu" "B.Cu") (free) (net 1))
   (via (at 78 70.5) (size 0.8) (drill 0.4) (layers "F.Cu" "B.Cu") (free) (net 1))
@@
   (via (at 106.2 133.2) (size 0.8) (drill 0.4) (layers "F.Cu" "B.Cu") (free) (net 1))
   (via (at 116.8 113.6) (size 0.8) (drill 0.4) (layers "F.Cu" "B.Cu") (free) (net 1))
+  (via (at 135.5 86.8) (size 0.8) (drill 0.4) (layers "F.Cu" "B.Cu") (free) (net 1))
   (via (at 115.6 124.4) (size 0.8) (drill 0.4) (layers "F.Cu" "B.Cu") (free) (net 1))
   (via (at 95.6 114.2) (size 0.8) (drill 0.4) (layers "F.Cu" "B.Cu") (free) (net 1))
@@
   (via (at 119.2 152) (size 0.8) (drill 0.4) (layers "F.Cu" "B.Cu") (free) (net 1))
   (via (at 57.6 136) (size 0.8) (drill 0.4) (layers "F.Cu" "B.Cu") (free) (net 1))
+  (via (at 127.9 79.2) (size 0.8) (drill 0.4) (layers "F.Cu" "B.Cu") (free) (net 1))
   (via (at 57 140.2) (size 0.8) (drill 0.4) (layers "F.Cu" "B.Cu") (free) (net 1))
   (via (at 68.6 152) (size 0.8) (drill 0.4) (layers "F.Cu" "B.Cu") (free) (net 1))
@@
   (segment (start 82 134.5) (end 82 130.5) (width 0.5) (layer "F.Cu") (net 49))
   (segment (start 92 127) (end 97.1165 121.8835) (width 0.5) (layer "F.Cu") (net 49))
-  (segment (start 82 129) (end 82.5 128.5) (width 0.5) (layer "F.Cu") (net 49))
   (segment (start 97.1165 121.8835) (end 97.959 121.8835) (width 0.5) (layer "F.Cu") (net 49))
   (segment (start 84.5 127) (end 92 127) (width 0.5) (layer "F.Cu") (net 49))
