File: circuito/rasp-sense33/trekking.kicad_sch (KiCad schematic)
At the start: 56 parts, among them J1 Raspberry Pi, J10 MOTOR, J11 OUT, J12 I2C0, J13 I2C0, J14 I2C0, J15 I2C0, J16 I2C0, J17 I2C0, J18 Module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

Commit message: correção medidor/mostrador, add media movel e offset
Other:
- note added: "0.15"
