File: circuito/PECDR-W/PECDR.kicad_sch (KiCad schematic)
At the start: 65 parts, among them J1 O2, J10 GP-SPI, J11 GP-SPI, J12 O3, J13 GND, J14 A, J15 B, J16 VS-SELECT, J17 GP-I2C1, J2 O4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

Commit message: PECDR update
Other:
- moved on the sheet: JP1, R5

Commit message: anotando correções em PECDR-W e criando programa de testes
Connections:
- net DriverInput: now also U3.21 (GP16); no longer U3.22 (GP17)
- net ReceiverOutput: now also U3.22 (GP17); no longer U3.21 (GP16)

Commit message: PECDR correção rs485 e de layout
Parts:
- R1: value 120 -> 4k7
Connections:
- net A: now also R1.1, R2.2; no longer R1.2, R3.1
- net B: now also R1.2, R3.1; no longer R1.1, R2.2
Changed lines of the file:
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@@
     (effects (font (size 1.27 1.27)) (justify right bottom))
   )
-  (label "B" (at 165.735 163.195 0) (fields_autoplaced)
+  (label "B" (at 165.735 170.815 0) (fields_autoplaced)
     (effects (font (size 1.27 1.27)) (justify left bottom))
   )
@@
     (effects (font (size 1.27 1.27)) (justify right bottom))
   )
-  (label "A" (at 165.735 170.815 0) (fields_autoplaced)
+  (label "A" (at 165.735 163.195 0) (fields_autoplaced)
     (effects (font (size 1.27 1.27)) (justify left bottom))
   )
@@
   (symbol (lib_id "Device:R") (at 153.67 167.005 0) (unit 1)
     (in_bom yes) (on_board yes) (dnp no) (fields_autoplaced)
-    (property "Reference" "R1" (at 155.575 165.735 0)
+    (property "Reference" "R1" (at 156.21 165.735 0)
       (effects (font (size 1.27 1.27)) (justify left))
     )
-    (property "Value" "120" (at 155.575 168.275 0)
+    (property "Value" "4k7" (at 156.21 168.275 0)
       (effects (font (size 1.27 1.27)) (justify left))
     )
